Commit message: Rebase from 'upstream'

File: kortex_description/arms/gen3/6dof/urdf/gen3_macro.xacro (robot description, xacro)
@@ -3,4 +3,5 @@
   <!-- Propagate last link name information because it is the gripper's parent link -->
   <xacro:property name="last_arm_link" value="end_effector_link"/>
+  <xacro:property name="PI" value="3.1415926535897931"/>
   <xacro:macro name="load_arm" params="
     parent
@@ -17,4 +18,7 @@
     connection_inactivity_timeout_ms:=2000
     use_internal_bus_gripper_comm:=false
+    gripper_joint_name
+    gripper_max_velocity:=100.0
+    gripper_max_force:=100.0
     use_fake_hardware:=false
     fake_sensor_commands:=false
@@ -22,4 +26,5 @@
     sim_ignition:=false
     sim_isaac:=false
+    use_external_cable:=false
     initial_positions:=${dict(joint_1=0.0,joint_2=0.0,joint_3=0.0,joint_4=0.0,joint_5=0.0,joint_6=0.0)}" >
     <!-- ros2 control include -->
@@ -41,5 +46,8 @@
       session_inactivity_timeout_ms="${session_inactivity_timeout_ms}"
       connection_inactivity_timeout_ms="${connection_inactivity_timeout_ms}"
-      use_internal_bus_gripper_comm="${use_internal_bus_gripper_comm}" />
+      use_internal_bus_gripper_comm="${use_internal_bus_gripper_comm}"
+      gripper_max_velocity="${gripper_max_velocity}"
+      gripper_max_force="${gripper_max_force}"
+      gripper_joint_name="${gripper_joint_name}"/>
     <joint name="${prefix}base_joint" type="fixed">
       <xacro:insert_block name="origin" />
@@ -91,17 +99,36 @@
       </collision>
     </link>
-    <joint
-      name="${prefix}joint_1"
-      type="continuous">
-      <origin
-        xyz="0 0 0.15643"
-        rpy="-3.1416 0.0 0.0" />
-      <parent link="${prefix}base_link" />
-      <child link="${prefix}shoulder_link" />
-      <axis xyz="0 0 1" />
-      <limit
-        effort="39"
-        velocity="1.3963" />
-    </joint>
+    <xacro:if value="${use_external_cable}">
+      <joint
+        name="${prefix}joint_1"
+        type="revolute">
+        <origin
+          xyz="0 0 0.15643"
+          rpy="-3.1416 0.0 0.0" />
+        <parent link="${prefix}base_link" />
+        <child link="${prefix}shoulder_link" />
+        <axis xyz="0 0 1" />
+        <limit
+          lower="${-2*PI}"
+          upper="${2*PI}"
+          effort="39"
+          velocity="1.3963" />
+      </joint>
+    </xacro:if>
+    <xacro:unless value="${use_external_cable}">
+      <joint
+        name="${prefix}joint_1"
+        type="continuous">
+        <origin
+          xyz="0 0 0.15643"
+          rpy="-3.1416 0.0 0.0" />
+        <parent link="${prefix}base_link" />
+        <child link="${prefix}shoulder_link" />
+        <axis xyz="0 0 1" />
+        <limit
+          effort="39"
+          velocity="1.3963" />
+      </joint>
+    </xacro:unless>
     <link name="${prefix}bicep_link">
       <inertial>
@@ -196,11 +223,22 @@
       </collision>
     </link>
-    <joint name="${prefix}joint_4" type="continuous">
-      <origin xyz="0 0.20843 -0.006375" rpy="1.5708 0.0 0.0" />
-      <parent link="${prefix}forearm_link" />
-      <child link="${prefix}spherical_wrist_1_link" />
-      <axis xyz="0 0 1" />
-      <limit effort="9" velocity="1.2218" />
-    </joint>
+    <xacro:if value="${use_external_cable}">
+      <joint name="${prefix}joint_4" type="revolute">
+        <origin xyz="0 0.20843 -0.006375" rpy="1.5708 0.0 0.0" />
+        <parent link="${prefix}forearm_link" />
+        <child link="${prefix}spherical_wrist_1_link" />
+        <axis xyz="0 0 1" />
+        <limit lower="${-2*PI}" upper="${2*PI}" effort="9" velocity="1.2218" />
+      </joint>
+    </xacro:if>
+    <xacro:unless value="${use_external_cable}">
+      <joint name="${prefix}joint_4" type="continuous">
+        <origin xyz="0 0.20843 -0.006375" rpy="1.5708 0.0 0.0" />
+        <parent link="${prefix}forearm_link" />
+        <child link="${prefix}spherical_wrist_1_link" />
+        <axis xyz="0 0 1" />
+        <limit effort="9" velocity="1.2218" />
+      </joint>
+    </xacro:unless>
     <link name="${prefix}spherical_wrist_2_link">
       <inertial>
@@ -280,11 +318,22 @@
     </link>
     </xacro:unless>
-    <joint name="${prefix}joint_6" type="continuous">
-      <origin xyz="0 0.10593 -0.00017505" rpy="1.5708 0.0 0.0" />
-      <parent link="${prefix}spherical_wrist_2_link" />
-      <child link="${prefix}bracelet_link" />
-      <axis xyz="0 0 1" />
-      <limit effort="9" velocity="1.2218" />
-    </joint>
+    <xacro:if value="${use_external_cable}">
+      <joint name="${prefix}joint_6" type="revolute">
+        <origin xyz="0 0.10593 -0.00017505" rpy="1.5708 0.0 0.0" />
+        <parent link="${prefix}spherical_wrist_2_link" />
+        <child link="${prefix}bracelet_link" />
+        <axis xyz="0 0 1" />
+        <limit lower="${-2*PI}" upper="${2*PI}" effort="9" velocity="1.2218" />
+      </joint>
+    </xacro:if>
+    <xacro:unless value="${use_external_cable}">
+      <joint name="${prefix}joint_6" type="continuous">
+        <origin xyz="0 0.10593 -0.00017505" rpy="1.5708 0.0 0.0" />
+        <parent link="${prefix}spherical_wrist_2_link" />
+        <child link="${prefix}bracelet_link" />
+        <axis xyz="0 0 1" />
+        <limit effort="9" velocity="1.2218" />
+      </joint>
+    </xacro:unless>
     <link name="${prefix}end_effector_link" />
     <joint

File: kortex_description/arms/gen3/7dof/urdf/gen3_macro.xacro (robot description, xacro)
@@ -26,4 +26,5 @@
     sim_ignition:=false
     sim_isaac:=false
+    use_external_cable:=false
     initial_positions:=${dict(joint_1=0.0,joint_2=0.0,joint_3=0.0,joint_4=0.0,joint_5=0.0,joint_6=0.0,joint_7=0.0)}" >
     <!-- ros2 control include -->
@@ -98,18 +99,38 @@
       </collision>
     </link>
-    <joint
+    <xacro:if value="${use_external_cable}">
+      <joint
       name="${prefix}joint_1"
-      type="continuous">
-      <origin xyz="0 0 0.15643" rpy="3.1416 2.7629E-18 -4.9305E-36" />
-      <parent
-        link="${prefix}base_link" />
-      <child
-        link="${prefix}shoulder_link" />
-      <axis
-        xyz="0 0 1" />
-      <limit
-        effort="39"
-        velocity="1.3963" />
-    </joint>
+      type="revolute">
+        <origin xyz="0 0 0.15643" rpy="3.1416 2.7629E-18 -4.9305E-36" />
+        <parent
+          link="${prefix}base_link" />
+        <child
+          link="${prefix}shoulder_link" />
+        <axis
+          xyz="0 0 1" />
+        <limit
+          lower="${-2*PI}"
+          upper="${2*PI}"
+          effort="39"
+          velocity="1.3963" />
+      </joint>
+    </xacro:if>
+    <xacro:unless value="${use_external_cable}">
+      <joint
+        name="${prefix}joint_1"
+        type="continuous">
+        <origin xyz="0 0 0.15643" rpy="3.1416 2.7629E-18 -4.9305E-36" />
+        <parent
+          link="${prefix}base_link" />
+        <child
+          link="${prefix}shoulder_link" />
+        <axis
+          xyz="0 0 1" />
+        <limit
+          effort="39"
+          velocity="1.3963" />
+      </joint>
+    </xacro:unless>
     <link name="${prefix}half_arm_1_link">
       <inertial>
@@ -168,18 +189,38 @@
       </collision>
     </link>
-    <joint
-      name="${prefix}joint_3"
-      type="continuous">
-      <origin xyz="0 -0.21038 -0.006375" rpy="-1.5708 1.2326E-32 -2.9122E-16" />
-      <parent
-        link="${prefix}half_arm_1_link" />
-      <child
-        link="${prefix}half_arm_2_link" />
-      <axis
-        xyz="0 0 1" />
-      <limit
-        effort="39"
-        velocity="1.3963" />
-    </joint>
+    <xacro:if value="${use_external_cable}">
+      <joint
+        name="${prefix}joint_3"
+        type="revolute">
+        <origin xyz="0 -0.21038 -0.006375" rpy="-1.5708 1.2326E-32 -2.9122E-16" />
+        <parent
+          link="${prefix}half_arm_1_link" />
+        <child
+          link="${prefix}half_arm_2_link" />
+        <axis
+          xyz="0 0 1" />
+        <limit
+          lower="${-2*PI}"
+          upper="${2*PI}"
+          effort="39"
+          velocity="1.3963" />
+      </joint>
+    </xacro:if>
+    <xacro:unless value="${use_external_cable}">
+      <joint
+        name="${prefix}joint_3"
+        type="continuous">
+        <origin xyz="0 -0.21038 -0.006375" rpy="-1.5708 1.2326E-32 -2.9122E-16" />
+        <parent
+          link="${prefix}half_arm_1_link" />
+        <child
+          link="${prefix}half_arm_2_link" />
+        <axis
+          xyz="0 0 1" />
+        <limit
+          effort="39"
+          velocity="1.3963" />
+      </joint>
+    </xacro:unless>
     <link name="${prefix}forearm_link">
       <inertial>
@@ -238,18 +279,38 @@
       </collision>
     </link>
-    <joint
-      name="${prefix}joint_5"
-      type="continuous">
-      <origin xyz="0 -0.20843 -0.006375" rpy="-1.5708 2.2204E-16 -6.373E-17" />
-      <parent
-        link="${prefix}forearm_link" />
-      <child
-        link="${prefix}spherical_wrist_1_link" />
-      <axis
-        xyz="0 0 1" />
-      <limit
-        effort="9"
-        velocity="1.2218" />
-    </joint>
+    <xacro:if value="${use_external_cable}">
+      <joint
+        name="${prefix}joint_5"
+        type="revolute">
+        <origin xyz="0 -0.20843 -0.006375" rpy="-1.5708 2.2204E-16 -6.373E-17" />
+        <parent
+          link="${prefix}forearm_link" />
+        <child
+          link="${prefix}spherical_wrist_1_link" />
+        <axis
+          xyz="0 0 1" />
+        <limit
+          lower="${-2*PI}"
+          upper="${2*PI}"
+          effort="9"
+          velocity="1.2218" />
+      </joint>
+    </xacro:if>
+    <xacro:unless value="${use_external_cable}">
+      <joint
+        name="${prefix}joint_5"
+        type="continuous">
+        <origin xyz="0 -0.20843 -0.006375" rpy="-1.5708 2.2204E-16 -6.373E-17" />
+        <parent
+          link="${prefix}forearm_link" />
+        <child
+          link="${prefix}spherical_wrist_1_link" />
+        <axis
+          xyz="0 0 1" />
+        <limit
+          effort="9"
+          velocity="1.2218" />
+      </joint>
+    </xacro:unless>
     <link name="${prefix}spherical_wrist_2_link">
       <inertial>
@@ -334,18 +395,38 @@
     </link>
     </xacro:unless>
-    <joint
-      name="${prefix}joint_7"
-      type="continuous">
-      <origin xyz="0 -0.10593 -0.00017505" rpy="-1.5708 -5.5511E-17 9.6396E-17" />
-      <parent
-        link="${prefix}spherical_wrist_2_link" />
-      <child
-        link="${prefix}bracelet_link" />
-      <axis
-        xyz="0 0 1" />
-      <limit
-        effort="9"
-        velocity="1.2218" />
-    </joint>
+    <xacro:if value="${use_external_cable}">
+      <joint
+        name="${prefix}joint_7"
+        type="revolute">
+        <origin xyz="0 -0.10593 -0.00017505" rpy="-1.5708 -5.5511E-17 9.6396E-17" />
+        <parent
+          link="${prefix}spherical_wrist_2_link" />
+        <child
+          link="${prefix}bracelet_link" />
+        <axis
+          xyz="0 0 1" />
+        <limit
+          lower="${-2*PI}"
+          upper="${2*PI}"
+          effort="9"
+          velocity="1.2218" />
+      </joint>
+    </xacro:if>
+    <xacro:unless value="${use_external_cable}">
+      <joint
+        name="${prefix}joint_7"
+        type="continuous">
+        <origin xyz="0 -0.10593 -0.00017505" rpy="-1.5708 -5.5511E-17 9.6396E-17" />
+        <parent
+          link="${prefix}spherical_wrist_2_link" />
+        <child
+          link="${prefix}bracelet_link" />
+        <axis
+          xyz="0 0 1" />
+        <limit
+          effort="9"
+          velocity="1.2218" />
+      </joint>
+    </xacro:unless>
     <link name="${prefix}end_effector_link" />
     <joint

File: kortex_description/robots/gen3.xacro (robot description, xacro)
@@ -23,4 +23,5 @@
     <xacro:arg name="fake_sensor_commands" default="false" />
     <xacro:arg name="use_internal_bus_gripper_comm" default="false" />
+    <xacro:arg name="use_external_cable" default="false" />
     <xacro:include filename="$(find kortex_description)/robots/kortex_robot.xacro" />
     <link name="world" />
@@ -47,5 +48,6 @@
         sim_gazebo="$(arg sim_gazebo)"
         sim_ignition="$(arg sim_ignition)"
-        sim_isaac="$(arg sim_isaac)" >
+        sim_isaac="$(arg sim_isaac)"
+        use_external_cable="$(arg use_external_cable)" >
         <origin xyz="0 0 0" rpy="0 0 0" />  <!-- position robot in the world -->
     </xacro:load_robot>

File: kortex_description/robots/kortex_robot.xacro (robot description, xacro)
@@ -23,4 +23,5 @@
     sim_ignition:=false
     sim_isaac:=false
+    use_external_cable:=false
     gripper_max_velocity:=100.0
     gripper_max_force:=100.0">
@@ -48,5 +49,6 @@
       gripper_joint_name="${gripper_joint_name}"
       gripper_max_velocity="${gripper_max_velocity}"
-      gripper_max_force="${gripper_max_force}">
+      gripper_max_force="${gripper_max_force}"
+      use_external_cable="${use_external_cable}">
       <xacro:insert_block name="origin" />
     </xacro:load_arm>
